File: Hardware/test_samd11/test_samd11/test_samd11.sch (KiCad schematic (older format))
At the start: 147 parts, among them J1 Conn_01x05_Female, U1 ATSAMD11C14A-SS

Commit message: fixed charlie plexed array
Connections:
- net at D1.2 (A), D101.2 (A), D112.2 (A)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: now also D12.1 (K), D13.1 (K), D14.1 (K), D15.1 (K), D16.1 (K), D17.1 (K), D18.1 (K), D19.1 (K), D20.1 (K), D21.1 (K), D22.1 (K), R2.1
- net at D102.2 (A), D113.2 (A), D124.2 (A)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: now also D23.1 (K), D24.1 (K), D25.1 (K), D26.1 (K), D27.1 (K), D28.1 (K), D29.1 (K), D30.1 (K), D31.1 (K), D32.1 (K), D33.1 (K), R3.1
- net at D103.2 (A), D114.2 (A), D125.2 (A)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: now also D34.1 (K), D35.1 (K), D36.1 (K), D37.1 (K), D38.1 (K), D39.1 (K), D40.1 (K), D41.1 (K), D42.1 (K), D43.1 (K), D44.1 (K), R4.1
- net at D104.2 (A), D115.2 (A), D126.2 (A)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: now also D45.1 (K), D46.1 (K), D47.1 (K), D48.1 (K), D49.1 (K), D50.1 (K), D51.1 (K), D52.1 (K), D53.1 (K), D54.1 (K), D55.1 (K), R5.1
- net at D105.2 (A), D116.2 (A), D127.2 (A)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: now also D56.1 (K), D57.1 (K), D58.1 (K), D59.1 (K), D60.1 (K), D61.1 (K), D62.1 (K), D63.1 (K), D64.1 (K), D65.1 (K), D66.1 (K), R6.1
- net at D106.2 (A), D117.2 (A), D128.2 (A)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: now also D67.1 (K), D68.1 (K), D69.1 (K), D70.1 (K), D71.1 (K), D72.1 (K), D73.1 (K), D74.1 (K), D75.1 (K), D76.1 (K), D77.1 (K), R7.1
- net at D107.2 (A), D118.2 (A), D129.2 (A)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: now also D78.1 (K), D79.1 (K), D80.1 (K), D81.1 (K), D82.1 (K), D83.1 (K), D84.1 (K), D85.1 (K), D86.1 (K), D87.1 (K), D88.1 (K), R8.1
- net at D108.2 (A), D119.2 (A), D130.2 (A)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: now also D89.1 (K), D90.1 (K), D91.1 (K), D92.1 (K), D93.1 (K), D94.1 (K), D95.1 (K), D96.1 (K), D97.1 (K), D98.1 (K), D99.1 (K), R9.1
- net at D120.2 (A), D131.2 (A), D20.2 (A)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: now also D100.1 (K), D101.1 (K), D102.1 (K), D103.1 (K), D104.1 (K), D105.1 (K), D106.1 (K), D107.1 (K), D108.1 (K), D109.1 (K), D110.1 (K), R10.1
- net at D10.2 (A), D109.2 (A), D132.2 (A)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: now also D111.1 (K), D112.1 (K), D113.1 (K), D114.1 (K), D115.1 (K), D116.1 (K), D117.1 (K), D118.1 (K), D119.1 (K), D120.1 (K), D121.1 (K), R11.1
Changed lines of the file:
@@
 EESchema Schematic File Version 4
+LIBS:test_samd11-cache
 EELAYER 29 0
 EELAYER END
@@
 Connection ~ 1500 1350
 Wire Wire Line
-	1500 1350 2000 1350
+	1500 1350 1800 1350
 Connection ~ 2000 1350
 Wire Wire Line
@@
 Connection ~ 2000 1850
 Wire Wire Line
-	2000 1850 2500 1850
+	2000 1850 2300 1850
 Connection ~ 2500 1850
 Wire Wire Line
@@
 Connection ~ 2500 2350
 Wire Wire Line
-	2500 2350 3000 2350
+	2500 2350 2800 2350
 Connection ~ 3000 2350
 Wire Wire Line
@@
 Connection ~ 3000 2850
 Wire Wire Line
-	3000 2850 3500 2850
+	3000 2850 3300 2850
 Connection ~ 3500 2850
 Wire Wire Line
@@
 Connection ~ 3500 3350
 Wire Wire Line
-	3500 3350 4000 3350
+	3500 3350 3800 3350
 Connection ~ 4000 3350
 Wire Wire Line
@@
 Connection ~ 4000 3850
 Wire Wire Line
-	4000 3850 4500 3850
+	4000 3850 4300 3850
 Connection ~ 4500 3850
 Wire Wire Line
@@
 Connection ~ 4500 4350
 Wire Wire Line
-	4500 4350 5000 4350
+	4500 4350 4800 4350
 Connection ~ 5000 4350
 Wire Wire Line
@@
 Connection ~ 5000 4850
 Wire Wire Line
-	5000 4850 5500 4850
+	5000 4850 5300 4850
 Connection ~ 5500 4850
 Wire Wire Line
@@
 Connection ~ 5500 5350
 Wire Wire Line
-	5500 5350 6000 5350
+	5500 5350 5800 5350
 Connection ~ 6000 5350
 Wire Wire Line
@@
 Connection ~ 6000 5850
 Wire Wire Line
-	6000 5850 6500 5850
-Wire Wire Line
 	1150 6350 1500 6350
 Connection ~ 1500 6350
@@
 	6000 6350 6500 6350
 Wire Wire Line
-	1800 1150 1800 2150
+	1800 1150 1800 1350
 Wire Wire Line
 	1800 6800 2000 6800
@@
 Connection ~ 6300 5650
 Wire Wire Line
-	6300 5650 6300 6800
+	6300 5650 6300 5850
 Wire Wire Line
 	5500 5150 5800 5150
 Connection ~ 5800 5150
 Wire Wire Line
-	5800 5150 5800 6150
+	5800 5150 5800 5350
 Wire Wire Line
 	5000 4650 5300 4650
 Connection ~ 5300 4650
 Wire Wire Line
-	5300 4650 5300 5650
+	5300 4650 5300 4850
 Wire Wire Line
 	4500 4150 4800 4150
@@
 Connection ~ 4300 3650
 Wire Wire Line
-	4300 3650 4300 4650
+	4300 3650 4300 3850
 Wire Wire Line
 	3500 3150 3800 3150
 Connection ~ 3800 3150
 Wire Wire Line
-	3800 3150 3800 4150
+	3800 3150 3800 3350
 Wire Wire Line
 	3000 2650 3300 2650
 Connection ~ 3300 2650
 Wire Wire Line
-	3300 2650 3300 3650
+	3300 2650 3300 2850
 Wire Wire Line
 	2500 2150 2800 2150
 Connection ~ 2800 2150
 Wire Wire Line
-	2800 2150 2800 3150
+	2800 2150 2800 2350
 Wire Wire Line
 	2000 1650 2300 1650
 Connection ~ 2300 1650
 Wire Wire Line
-	2300 1650 2300 2650
+	2300 1650 2300 1850
 Wire Wire Line
 	1300 850  1300 1650
@@
 	5000 5150 4800 5150
 Wire Wire Line
-	4800 4150 4800 5150
+	4800 4150 4800 4350
 Connection ~ 4800 5150
 Wire Wire Line
@@
 Text GLabel 10600 3150 2    50   Input ~ 0
 LED12
+Wire Wire Line
+	6000 5850 6300 5850
+Connection ~ 6300 5850
+Wire Wire Line
+	6300 5850 6300 6800
+Wire Wire Line
+	6300 5850 6500 5850
+Wire Wire Line
+	6000 5350 5800 5350
+Connection ~ 5800 5350
+Wire Wire Line
+	5800 5350 5800 6150
+Wire Wire Line
+	5500 4850 5300 4850
+Connection ~ 5300 4850
+Wire Wire Line
+	5300 4850 5300 5650
+Wire Wire Line
+	5000 4350 4800 4350
+Connection ~ 4800 4350
+Wire Wire Line
+	4800 4350 4800 5150
+Wire Wire Line
+	4500 3850 4300 3850
+Connection ~ 4300 3850
+Wire Wire Line
+	4300 3850 4300 4650
+Wire Wire Line
+	4000 3350 3800 3350
+Connection ~ 3800 3350
+Wire Wire Line
+	3800 3350 3800 4150
+Wire Wire Line
+	3500 2850 3300 2850
+Connection ~ 3300 2850
+Wire Wire Line
+	3300 2850 3300 3650
+Wire Wire Line
+	3000 2350 2800 2350
+Connection ~ 2800 2350
+Wire Wire Line
+	2800 2350 2800 3150
+Wire Wire Line
+	2500 1850 2300 1850
+Connection ~ 2300 1850
+Wire Wire Line
+	2300 1850 2300 2650
+Wire Wire Line
+	2000 1350 1800 1350
+Connection ~ 1800 1350
+Wire Wire Line
+	1800 1350 2000 1350
+Wire Wire Line
+	1800 1350 1800 2150
 $EndSCHEMATC
