File: Hardware/kicad_project/tdm_v6.kicad_pcb (KiCad board)
At the start: 4 copper layers, 65 x 100 mm, 214 parts, among them J1 picoprobe_debug, J2 USB_C_Receptacle_USB2.0, J3 line_in, J4 headphone_out, J5 midi_in, J6 midi_out, J7 battery, J8 Conn_01x03_Male, Q1 DMG2305UX-13, Q2 Q_PMOS_GSD, Q3 Q_NMOS_GSD, Q4 Q_NMOS_GSD, SW1 spst_4_pin_internal, SW10 spst_4_pin_internal, SW11 spst_4_pin_internal, SW12 spst_4_pin_internal, SW13 spst_4_pin_internal, SW14 spst_4_pin_internal, SW15 spst_4_pin_internal, SW16 spst_4_pin_internal, SW17 spst_4_pin_internal, SW18 spst_4_pin_internal, SW19 spst_4_pin_internal, SW2 spst_4_pin_internal, SW20 spst_4_pin_internal, SW21 spst_4_pin_internal, SW22 spst_4_pin_internal, SW23 spst_4_pin_internal, SW24 spst_4_pin_internal, SW25 spst_4_pin_internal, SW26 spst_4_pin_internal, SW27 spst_4_pin_internal, SW3 spst_4_pin_internal, SW4 spst_4_pin_internal, SW5 spst_4_pin_internal, SW6 spst_4_pin_internal, SW7 spst_4_pin_internal, SW8 spst_4_pin_internal, SW9 spst_4_pin_internal, U1 W25Q32JVSS, U10 apx804SR, U11 ME6211C, U2 RP2040, U3 TLV320AIC3204, U4 AP3722AT_mic, U5 6N137, U6 MCP73831T-2ATI_OT, U7 apx804SR, U8 LM4890, U9 ME6211C, Y1 Crystal_GND24

Commit message: v9 hardware
Parts:
- removed C66: 1u, Capacitors_Tantalum_SMD:CP_Tantalum_Case-A_EIA-3216-18_Reflow
- removed C67: 470nf, Capacitors_Tantalum_SMD:CP_Tantalum_Case-A_EIA-3216-18_Reflow
- removed J8: Conn_01x03_Male, Connector_PinHeader_2.54mm:PinHeader_1x03_P2.54mm_Horizontal
- removed LS1: Speaker, Connector_PinHeader_2.54mm:PinHeader_1x02_P2.54mm_Horizontal
- removed U10, U7: apx804SR, TO_SOT_Packages_SMD:SOT-23
- removed U8: LM4890, Housings_SSOP:MSOP-8_3x3mm_Pitch0.65mm
- added D26: D_Zener, Diode_SMD:D_SOD-323, F.Cu at (80.5, 40.5)
- added D3: D_Zener, Diode_SMD:D_SOD-323, F.Cu at (91.0, 46.0)
- added D4: D_Zener, Diode_SMD:D_SOD-323, F.Cu at (89.0, 46.0)
- added D5: D_Zener, Diode_SMD:D_SOD-323, F.Cu at (78.5, 40.5)
- added J9: Conn_01x02_Female, Connector_PinHeader_2.54mm:PinHeader_1x02_P2.54mm_Vertical, F.Cu at (36.7, 90.0)
- added JP10: SolderJumper_2_Open, Jumper:SolderJumper-2_P1.3mm_Open_RoundedPad1.0x1.5mm, B.Cu at (40.6, 77.1)
- added JP11: SolderJumper_2_Open, Jumper:SolderJumper-2_P1.3mm_Open_RoundedPad1.0x1.5mm, B.Cu at (50.0, 80.5)
- added JP12: SolderJumper_2_Open, Jumper:SolderJumper-2_P1.3mm_Open_RoundedPad1.0x1.5mm, B.Cu at (36.8, 96.2)
- added JP13: SolderJumper_2_Bridged, Jumper:SolderJumper-2_P1.3mm_Bridged_Pad1.0x1.5mm, B.Cu at (43.2, 80.5)
- added JP14: SolderJumper_2_Bridged, Jumper:SolderJumper-2_P1.3mm_Bridged_Pad1.0x1.5mm, B.Cu at (37.3, 123.4)
- added JP15: SolderJumper_2_Bridged, Jumper:SolderJumper-2_P1.3mm_Bridged_Pad1.0x1.5mm, B.Cu at (85.1, 45.7)
- added JP16: SolderJumper_2_Open, Jumper:SolderJumper-2_P1.3mm_Open_RoundedPad1.0x1.5mm, B.Cu at (86.9, 37.8)
- added JP17: SolderJumper_2_Open, Jumper:SolderJumper-2_P1.3mm_Open_RoundedPad1.0x1.5mm, B.Cu at (67.3, 35.2)
- added JP18: SolderJumper_2_Bridged, Jumper:SolderJumper-2_P1.3mm_Bridged_Pad1.0x1.5mm, B.Cu at (68.0, 41.5)
- added JP9: SolderJumper_2_Bridged, Jumper:SolderJumper-2_P1.3mm_Bridged_Pad1.0x1.5mm, B.Cu at (36.6, 79.1)
- added R32: 100, MyLibrary:LED_0402_nosilk, F.Cu at (87.0, 46.5)
- added R33: 100, MyLibrary:LED_0402_nosilk, F.Cu at (71.0, 41.0)
- C4: value 1u -> 10u; footprint Capacitors_Tantalum_SMD:CP_Tantalum_Case-A_EIA-3216-18_Reflow -> RandomJunk:C_0402_NoSilk
- C65: value 470nf -> 100u; footprint Capacitors_Tantalum_SMD:CP_Tantalum_Case-A_EIA-3216-18_Reflow -> Capacitor_Tantalum_SMD:CP_EIA-3528-21_Kemet-B
- D10, D11, D12, D13, D14, D15, D16, D17, D18, D19, D20, D21, D22, D23, D24, D25, D6, D7, D8, D9: value WS2812B -> WS2812C-v1
- JP7, JP8: value SolderJumper_2_Bridged -> SolderJumper_2_Open; footprint Jumper:SolderJumper-2_P1.3mm_Bridged_Pad1.0x1.5mm -> Jumper:SolderJumper-2_P1.3mm_Open_RoundedPad1.0x1.5mm
- R21: value 20k -> 10
- R22, R23, R30: value 20k -> 33
- SW1, SW10, SW11, SW12, SW13, SW14, SW15, SW16, SW17, SW18, SW19, SW2, SW20, SW21, SW22, SW23, SW24, SW25, SW3, SW4, SW5, SW6, SW7, SW8, SW9: footprint RandomJunk:ts1102_smallerpads_buttonhole -> MyLibrary:ts1187
- SW26, SW27: footprint RandomJunk:ts1102_smallerpads_buttonhole -> MyLibrary:SKSCLDE010; moved to F.Cu
- moved R21 64.2 mm to (37.2, 80.8)
- moved R22 64.0 mm to (38.5, 78.9)
- moved R30 63.6 mm to (38.5, 81.0), turned to 90 degrees
- moved C65 63.5 mm to (37.0, 86.2)
- moved JP8 62.8 mm to (40.5, 80.5), turned to -90 degrees
- moved R23 62.6 mm to (37.2, 78.9), turned to 90 degrees
- moved C4 62.5 mm to (37.4, 83.0)
- moved JP7 62.4 mm to (36.6, 82.5), turned to -90 degrees
- moved SW26 14.0 mm to (96.8, 45.0), turned to 90 degrees
- moved SW27 6.58 mm to (96.8, 50.5), turned to 90 degrees
- moved D28 4.99 mm to (65.8, 78.7), turned to 180 degrees
- moved D29 4.98 mm to (77.1, 78.7), turned to 180 degrees
- moved D30 4.93 mm to (87.8, 78.7), turned to 180 degrees
- moved D27 4.88 mm to (54.7, 78.7), turned to 180 degrees
- moved D31 4.88 mm to (43.7, 90.7), turned to 180 degrees
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Connections:
- C10 pad 1: +3V3 -> Net-(C10-Pad1)
- C10 pad 2: GND -> Net-(C10-Pad2)
- C11 pad 1: +3V3 -> Net-(C10-Pad1)
- C11 pad 2: GND -> Net-(C10-Pad2)
- C12 pad 1: +3V3 -> Net-(C10-Pad1)
- C12 pad 2: GND -> Net-(C10-Pad2)
- C13 pad 1: +3V3 -> Net-(C10-Pad1)
- C13 pad 2: GND -> Net-(C10-Pad2)
- C14 pad 1: +3V3 -> Net-(C10-Pad1)
- C14 pad 2: GND -> Net-(C10-Pad2)
- C15 pad 1: +3V3 -> Net-(C10-Pad1)
- C15 pad 2: GND -> Net-(C10-Pad2)
- C16 pad 1: +3V3 -> Net-(C10-Pad1)
- C16 pad 2: GND -> Net-(C10-Pad2)
- C17 pad 1: +3V3 -> Net-(C10-Pad1)
- C17 pad 2: GND -> Net-(C10-Pad2)
- C18 pad 1: +3V3 -> Net-(C10-Pad1)
- C18 pad 2: GND -> Net-(C10-Pad2)
- C19 pad 1: +3V3 -> Net-(C10-Pad1)
- C19 pad 2: GND -> Net-(C10-Pad2)
- C20 pad 1: +3V3 -> Net-(C10-Pad1)
- C20 pad 2: GND -> Net-(C10-Pad2)
- C21 pad 1: +3V3 -> Net-(C10-Pad1)
- C21 pad 2: GND -> Net-(C10-Pad2)
- C22 pad 1: +3V3 -> Net-(C10-Pad1)
- C22 pad 2: GND -> Net-(C10-Pad2)
- C23 pad 1: +3V3 -> Net-(C10-Pad1)
- C23 pad 2: GND -> Net-(C10-Pad2)
- C24 pad 1: +3V3 -> Net-(C10-Pad1)
- C24 pad 2: GND -> Net-(C10-Pad2)
- C25 pad 1: +3V3 -> Net-(C10-Pad1)
- C25 pad 2: GND -> Net-(C10-Pad2)
- C6 pad 1: +3V3 -> Net-(C10-Pad1)
- C6 pad 2: GND -> Net-(C10-Pad2)
- C65 pad 1: Net-(C65-Pad1) -> Net-(C4-Pad1)
- C65 pad 2: /AudioMidi/lineout_left -> GND
- C7 pad 1: +3V3 -> Net-(C10-Pad1)
- C7 pad 2: GND -> Net-(C10-Pad2)
- C8 pad 1: +3V3 -> Net-(C10-Pad1)
- C8 pad 2: GND -> Net-(C10-Pad2)
- C9 pad 1: +3V3 -> Net-(C10-Pad1)
- C9 pad 2: GND -> Net-(C10-Pad2)
- D10 pad 2: GND -> Net-(C10-Pad2)
- D10 pad 4: +3V3 -> Net-(C10-Pad1)
- D11 pad 2: GND -> Net-(C10-Pad2)
- D11 pad 4: +3V3 -> Net-(C10-Pad1)
- D12 pad 2: GND -> Net-(C10-Pad2)
- D12 pad 4: +3V3 -> Net-(C10-Pad1)
- D13 pad 2: GND -> Net-(C10-Pad2)
- D13 pad 4: +3V3 -> Net-(C10-Pad1)
- D14 pad 2: GND -> Net-(C10-Pad2)
- D14 pad 4: +3V3 -> Net-(C10-Pad1)
- D15 pad 2: GND -> Net-(C10-Pad2)
- D15 pad 4: +3V3 -> Net-(C10-Pad1)
- D16 pad 2: GND -> Net-(C10-Pad2)
- D16 pad 4: +3V3 -> Net-(C10-Pad1)
- D17 pad 2: GND -> Net-(C10-Pad2)
- D17 pad 4: +3V3 -> Net-(C10-Pad1)
- D18 pad 2: GND -> Net-(C10-Pad2)
- D18 pad 4: +3V3 -> Net-(C10-Pad1)
- D19 pad 2: GND -> Net-(C10-Pad2)
- D19 pad 4: +3V3 -> Net-(C10-Pad1)
- D20 pad 2: GND -> Net-(C10-Pad2)
- D20 pad 4: +3V3 -> Net-(C10-Pad1)
- D21 pad 2: GND -> Net-(C10-Pad2)
- D21 pad 4: +3V3 -> Net-(C10-Pad1)
- D22 pad 2: GND -> Net-(C10-Pad2)
- D22 pad 4: +3V3 -> Net-(C10-Pad1)
- D23 pad 2: GND -> Net-(C10-Pad2)
- D23 pad 4: +3V3 -> Net-(C10-Pad1)
- D24 pad 2: GND -> Net-(C10-Pad2)
- D24 pad 4: +3V3 -> Net-(C10-Pad1)
- D25 pad 1: Net-(D25-Pad1) -> unconnected-(D25-Pad1)
- D25 pad 2: GND -> Net-(C10-Pad2)
- D25 pad 4: +3V3 -> Net-(C10-Pad1)
- D6 pad 2: GND -> Net-(C10-Pad2)
- D6 pad 4: +3V3 -> Net-(C10-Pad1)
- D7 pad 2: GND -> Net-(C10-Pad2)
- D7 pad 4: +3V3 -> Net-(C10-Pad1)
- D8 pad 2: GND -> Net-(C10-Pad2)
- D8 pad 4: +3V3 -> Net-(C10-Pad1)
- D9 pad 2: GND -> Net-(C10-Pad2)
- D9 pad 4: +3V3 -> Net-(C10-Pad1)
- J2 pad A8: Net-(J2-PadA8) -> unconnected-(J2-PadA8)
- J2 pad B8: Net-(J2-PadB8) -> unconnected-(J2-PadB8)
- J3 pad 2: Net-(C39-Pad2) -> Net-(J3-Pad2)
- J3 pad 3: Net-(C44-Pad2) -> Net-(J3-Pad3)
- J5 pad 4: Net-(J5-Pad4) -> unconnected-(J5-Pad4)
- J6 pad 4: Net-(J6-Pad4) -> unconnected-(J6-Pad4)
- JP7 pad 1: Net-(C4-Pad1) -> +3V3
- JP7 pad 2: Net-(JP7-Pad2) -> Net-(J9-Pad1)
- JP8 pad 1: Net-(JP8-Pad1) -> +3V3
- LCD1 pad 6: Net-(LCD1-Pad6) -> unconnected-(LCD1-Pad6)
- R14 pad 1: +3V3A -> GND
- R21 pad 1: Net-(C65-Pad1) -> Net-(C4-Pad1)
- R21 pad 2: Net-(JP8-Pad1) -> Net-(JP8-Pad2)
- R22 pad 1: Net-(LS1-Pad2) -> Net-(C4-Pad1)
- R22 pad 2: Net-(R22-Pad2) -> Net-(JP9-Pad1)
- R23 pad 1: Net-(JP8-Pad2) -> Net-(C4-Pad1)
- R23 pad 2: Net-(JP7-Pad2) -> Net-(JP9-Pad1)
- R30 pad 1: Net-(C67-Pad1) -> Net-(C4-Pad1)
- R30 pad 2: Net-(R22-Pad2) -> Net-(JP10-Pad2)
- SW1 pad 2: Net-(SW1-Pad2) -> unconnected-(SW1-Pad2)
- SW1 pad 4: Net-(SW1-Pad4) -> unconnected-(SW1-Pad4)
- SW10 pad 2: Net-(SW10-Pad2) -> unconnected-(SW10-Pad2)
- SW11 pad 2: Net-(SW11-Pad2) -> unconnected-(SW11-Pad2)
- SW12 pad 2: Net-(SW12-Pad2) -> unconnected-(SW12-Pad2)
- SW13 pad 2: Net-(SW13-Pad2) -> unconnected-(SW13-Pad2)
- SW14 pad 2: Net-(SW14-Pad2) -> unconnected-(SW14-Pad2)
- SW15 pad 2: Net-(SW15-Pad2) -> unconnected-(SW15-Pad2)
- SW16 pad 2: Net-(SW16-Pad2) -> unconnected-(SW16-Pad2)
- SW17 pad 2: Net-(SW17-Pad2) -> unconnected-(SW17-Pad2)
- SW18 pad 2: Net-(SW18-Pad2) -> unconnected-(SW18-Pad2)
- SW19 pad 2: Net-(SW19-Pad2) -> unconnected-(SW19-Pad2)
- SW2 pad 2: Net-(SW2-Pad2) -> unconnected-(SW2-Pad2)
- SW20 pad 2: Net-(SW20-Pad2) -> unconnected-(SW20-Pad2)
- SW21 pad 2: Net-(SW21-Pad2) -> unconnected-(SW21-Pad2)
- SW21 pad 3: Net-(SW21-Pad3) -> unconnected-(SW21-Pad3)
- SW22 pad 2: Net-(SW22-Pad2) -> unconnected-(SW22-Pad2)
- SW22 pad 3: Net-(SW22-Pad3) -> unconnected-(SW22-Pad3)
- SW23 pad 2: Net-(SW23-Pad2) -> unconnected-(SW23-Pad2)
- SW23 pad 3: Net-(SW23-Pad3) -> unconnected-(SW23-Pad3)
- SW24 pad 2: Net-(SW24-Pad2) -> unconnected-(SW24-Pad2)
- SW24 pad 3: Net-(SW24-Pad3) -> unconnected-(SW24-Pad3)
- SW25 pad 2: Net-(SW25-Pad2) -> unconnected-(SW25-Pad2)
- SW25 pad 3: Net-(SW25-Pad3) -> unconnected-(SW25-Pad3)
- SW26 pad 1: Net-(SW26-Pad1) -> unconnected-(SW26-Pad1)
- SW26 pad 4: Net-(SW26-Pad4) -> unconnected-(SW26-Pad4)
- SW27 pad 2: Net-(SW27-Pad2) -> unconnected-(SW27-Pad2)
- SW27 pad 4: Net-(SW27-Pad4) -> unconnected-(SW27-Pad4)
- SW3 pad 2: Net-(SW3-Pad2) -> unconnected-(SW3-Pad2)
- SW4 pad 2: Net-(SW4-Pad2) -> unconnected-(SW4-Pad2)
- SW5 pad 2: Net-(SW5-Pad2) -> unconnected-(SW5-Pad2)
- SW6 pad 2: Net-(SW6-Pad2) -> unconnected-(SW6-Pad2)
- SW7 pad 2: Net-(SW7-Pad2) -> unconnected-(SW7-Pad2)
- SW8 pad 2: Net-(SW8-Pad2) -> unconnected-(SW8-Pad2)
- SW9 pad 2: Net-(SW9-Pad2) -> unconnected-(SW9-Pad2)
- U11 pad 4: Net-(U11-Pad4) -> unconnected-(U11-Pad4)
- U3 pad 11: Net-(U3-Pad11) -> unconnected-(U3-Pad11)
- U3 pad 20: Net-(U3-Pad20) -> unconnected-(U3-Pad20)
- U3 pad 21: Net-(U3-Pad21) -> unconnected-(U3-Pad21)
- U3 pad 31: Net-(U3-Pad31) -> Net-(JP3-Pad1)
- U3 pad 32: Net-(JP3-Pad1) -> unconnected-(U3-Pad32)
- U3 pad 8: Net-(U3-Pad8) -> unconnected-(U3-Pad8)
- U5 pad 1: Net-(U5-Pad1) -> unconnected-(U5-Pad1)
- U5 pad 4: Net-(U5-Pad4) -> unconnected-(U5-Pad4)
- U5 pad 7: Net-(U5-Pad7) -> unconnected-(U5-Pad7)
- U9 pad 4: Net-(U9-Pad4) -> unconnected-(U9-Pad4)
- Y1 pad 2: Net-(Y1-Pad2) -> unconnected-(Y1-Pad2)
- Y1 pad 4: Net-(Y1-Pad4) -> unconnected-(Y1-Pad4)
Routing:
- net Net-(C10-Pad2): track 0.00 -> 482.6 mm, vias 0 -> 80
- net Net-(C10-Pad1): track 0.00 -> 391.1 mm, vias 0 -> 23
- net +3V3: track 318.4 -> 192.2 mm, vias 43 -> 11
- net GND: track 266.1 -> 192.4 mm, vias 34 -> 24
- net Net-(LS1-Pad1): track 47.7 -> 0.00 mm
- net VBUS: track 69.6 -> 113.9 mm, vias 5 -> 8
- net amp_control: track 39.1 -> 0.00 mm, vias 2 -> 0
- net +3V3A: track 92.2 -> 53.9 mm, vias 5 -> 4
- net Net-(LS1-Pad2): track 28.0 -> 0.00 mm
- net Net-(R6-Pad2): track 30.4 -> 51.2 mm, vias 3 -> 2
- net Net-(J3-Pad3): track 0.00 -> 16.5 mm
- net Net-(SW10-Pad4): track 3.60 -> 18.9 mm, vias 0 -> 2
- net tx: track 91.9 -> 106.7 mm, vias 1 -> 2
- net Net-(SW10-Pad3): track 3.60 -> 17.4 mm, vias 0 -> 2
- net Net-(SW2-Pad3): track 6.22 -> 19.9 mm
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- removed copper zone on B.Cu, net +3V3
- removed copper zone on In2.Cu, net +3V3
- removed copper zone on In2.Cu, net +3V3A
- removed copper zone on In1.Cu, net GND
Other:
- rule pad_to_mask_clearance: 0.051 -> 0

Commit message: v10 board
Parts:
- removed D52: D, RandomJunk:D_SOD-323F_less_silk
- removed J9: Conn_01x02_Female, Connector_PinHeader_2.54mm:PinHeader_1x02_P2.54mm_Vertical
- removed JP10, JP11, JP12, JP16, JP17: SolderJumper_2_Open, Jumper:SolderJumper-2_P1.3mm_Open_RoundedPad1.0x1.5mm
- removed JP13, JP15, JP18, JP9: SolderJumper_2_Bridged, Jumper:SolderJumper-2_P1.3mm_Bridged_Pad1.0x1.5mm
- added C66: 2u2, MyLibrary:C_0402_1005Metric, F.Cu at (56.0, 42.5)
- added J8: Conn_01x02_Female, Connector_PinHeader_2.54mm:PinHeader_1x02_P2.54mm_Vertical, B.Cu at (36.6, 78.5)
- added R34: 33, MyLibrary:R_0402_1005Metric_nosilk, F.Cu at (39.1, 45.5)
- added R35: 33, MyLibrary:R_0402_1005Metric_nosilk, F.Cu at (39.1, 46.5)
- added U7: LM4040DBZ-2.5, Package_TO_SOT_SMD:SOT-23, F.Cu at (61.7, 41.4)
- C1, C10, C11, C12, C13, C14, C15, C16, C17, C18, C19, C2, C20, C21, C22, C23, C24, C25, C26, C27, C28, C29, C3, C30, C31, C32, C33, C34, C35, C36, C37, C38, C4, C40, C41, C42, C43, C46, C5, C50, C51, C52, C53, C54, C55, C56, C57, C59, C6, C60, C61, C62, C63, C64, C7, C8, C9: footprint RandomJunk:C_0402_NoSilk -> MyLibrary:C_0402_1005Metric
- D26, D3, D4, D5: footprint Diode_SMD:D_SOD-323 -> Diode_SMD:D_SOD-323F
- JP7, JP8: value SolderJumper_2_Open -> SolderJumper_2_Bridged; footprint Jumper:SolderJumper-2_P1.3mm_Open_RoundedPad1.0x1.5mm -> Jumper:SolderJumper-2_P1.3mm_Bridged_Pad1.0x1.5mm
- LCD1: footprint RandomJunk:oled_ssd1306_14pin_91 -> MyLibrary:oled_ssd1306_14pin_91
- R1, R10, R14, R15, R16, R17, R18, R19, R2, R20, R24, R25, R26, R27, R28, R3, R31, R4, R5, R6, R7, R8, R9: footprint RandomJunk:R_0402_NoSilk -> MyLibrary:R_0402_1005Metric_nosilk
- R11: value 1k -> 220; footprint RandomJunk:R_0402_NoSilk -> MyLibrary:R_0402_1005Metric_nosilk
- R12: value 220 -> 33; footprint RandomJunk:R_0402_NoSilk -> MyLibrary:R_0402_1005Metric_nosilk
- R13: value 220 -> 10; footprint RandomJunk:R_0402_NoSilk -> MyLibrary:R_0402_1005Metric_nosilk
- R21: value 10 -> 220; footprint RandomJunk:R_0402_NoSilk -> MyLibrary:R_0402_1005Metric_nosilk
- R22: value 33 -> 330; footprint RandomJunk:R_0402_NoSilk -> MyLibrary:R_0402_1005Metric_nosilk
- R23: value 33 -> 5k; footprint RandomJunk:R_0402_NoSilk -> MyLibrary:R_0402_1005Metric_nosilk
- R30: value 33 -> 10k; footprint RandomJunk:R_0402_NoSilk -> MyLibrary:R_0402_1005Metric_nosilk
- R32, R33: footprint MyLibrary:LED_0402_nosilk -> Resistor_SMD:R_0402_1005Metric
- U5: value 6N137 -> HCPL-0631; footprint RandomJunk:SOP-8_3.9x5.1x1.27P -> Package_SO:SOIC-8_3.9x4.9mm_P1.27mm
- moved R30 47.7 mm to (67.1, 42.8), turned to 180 degrees
- moved R23 47.6 mm to (67.1, 41.8), turned to 0 degrees
- moved C65 45.8 mm to (37.0, 40.5), turned to 0 degrees
- moved R22 42.7 mm to (57.7, 40.8)
- moved R21 33.4 mm to (37.1, 47.5), turned to -90 degrees
- moved JP8 31.1 mm to (38.1, 49.5), turned to 0 degrees
- moved JP7 30.5 mm to (38.1, 52.1), turned to 180 degrees
- moved C4 26.5 mm to (41.5, 56.9), turned to 0 degrees
- moved R11 9.82 mm to (40.6, 47.5), turned to -90 degrees
- moved C50 9.59 mm to (38.6, 47.5), turned to 0 degrees
- moved R10 7.43 mm to (43.5, 54.3)
- moved C33 4.61 mm to (56.0, 47.5), turned to 180 degrees
- moved C53 4.17 mm to (42.9, 70.1), turned to 0 degrees
- moved R1 2.40 mm to (53.9, 46.5)
- moved C52 2.30 mm to (39.6, 56.9)
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Connections:
- C10 pad 1: Net-(C10-Pad1) -> 3v3_filter
- C11 pad 1: Net-(C10-Pad1) -> 3v3_filter
- C12 pad 1: Net-(C10-Pad1) -> 3v3_filter
- C13 pad 1: Net-(C10-Pad1) -> 3v3_filter
- C14 pad 1: Net-(C10-Pad1) -> 3v3_filter
- C15 pad 1: Net-(C10-Pad1) -> 3v3_filter
- C16 pad 1: Net-(C10-Pad1) -> 3v3_filter
- C17 pad 1: Net-(C10-Pad1) -> 3v3_filter
- C18 pad 1: Net-(C10-Pad1) -> 3v3_filter
- C19 pad 1: Net-(C10-Pad1) -> 3v3_filter
- C20 pad 1: Net-(C10-Pad1) -> 3v3_filter
- C21 pad 1: Net-(C10-Pad1) -> 3v3_filter
- C22 pad 1: Net-(C10-Pad1) -> 3v3_filter
- C23 pad 1: Net-(C10-Pad1) -> 3v3_filter
- C24 pad 1: Net-(C10-Pad1) -> 3v3_filter
- C25 pad 1: Net-(C10-Pad1) -> 3v3_filter
- C4 pad 1: Net-(C4-Pad1) -> +3V3
- C50 pad 1: +3V3 -> Net-(C50-Pad1)
- C53 pad 1: +3V3 -> 3v3_filter
- C6 pad 1: Net-(C10-Pad1) -> 3v3_filter
- C65 pad 1: Net-(C4-Pad1) -> Net-(C50-Pad1)
- C7 pad 1: Net-(C10-Pad1) -> 3v3_filter
- C8 pad 1: Net-(C10-Pad1) -> 3v3_filter
- C9 pad 1: Net-(C10-Pad1) -> 3v3_filter
- D10 pad 4: Net-(C10-Pad1) -> 3v3_filter
- D11 pad 4: Net-(C10-Pad1) -> 3v3_filter
- D12 pad 4: Net-(C10-Pad1) -> 3v3_filter
- D13 pad 4: Net-(C10-Pad1) -> 3v3_filter
- D14 pad 4: Net-(C10-Pad1) -> 3v3_filter
- D15 pad 4: Net-(C10-Pad1) -> 3v3_filter
- D16 pad 4: Net-(C10-Pad1) -> 3v3_filter
- D17 pad 4: Net-(C10-Pad1) -> 3v3_filter
- D18 pad 4: Net-(C10-Pad1) -> 3v3_filter
- D19 pad 4: Net-(C10-Pad1) -> 3v3_filter
- D20 pad 4: Net-(C10-Pad1) -> 3v3_filter
- D21 pad 4: Net-(C10-Pad1) -> 3v3_filter
- D22 pad 4: Net-(C10-Pad1) -> 3v3_filter
- D23 pad 4: Net-(C10-Pad1) -> 3v3_filter
- D24 pad 4: Net-(C10-Pad1) -> 3v3_filter
- D25 pad 4: Net-(C10-Pad1) -> 3v3_filter
- D6 pad 4: Net-(C10-Pad1) -> 3v3_filter
- D7 pad 4: Net-(C10-Pad1) -> 3v3_filter
- D8 pad 4: Net-(C10-Pad1) -> 3v3_filter
- D9 pad 4: Net-(C10-Pad1) -> 3v3_filter
- J5 pad 2: Net-(D52-Pad2) -> Net-(J5-Pad2)
- JP7 pad 1: +3V3 -> Net-(JP7-Pad1)
- JP7 pad 2: Net-(J9-Pad1) -> Net-(C50-Pad1)
- JP8 pad 1: +3V3 -> Net-(C50-Pad1)
- JP8 pad 2: Net-(JP8-Pad2) -> 3v3_filter
- LCD1 pad 5: +3V3 -> 3v3_filter
- R10 pad 1: Net-(D52-Pad1) -> /MIDI_RX
- R10 pad 2: Net-(J5-Pad3) -> +3V3
- R11 pad 1: /MIDI_RX -> Net-(J5-Pad3)
- R11 pad 2: +3V3 -> Net-(R11-Pad2)
- R21 pad 1: Net-(C4-Pad1) -> Net-(J5-Pad2)
- R21 pad 2: Net-(JP8-Pad2) -> Net-(R21-Pad2)
- R22 pad 1: Net-(C4-Pad1) -> vref2.5
- R22 pad 2: Net-(JP9-Pad1) -> VBUS
- R23 pad 1: Net-(C4-Pad1) -> usb_sense
- R23 pad 2: Net-(JP9-Pad1) -> VBUS
- R30 pad 1: Net-(C4-Pad1) -> GND
- R30 pad 2: Net-(JP10-Pad2) -> usb_sense
- R32 pad 2: Net-(JP15-Pad1) -> Net-(J3-Pad2)
- R33 pad 2: Net-(JP18-Pad1) -> Net-(J3-Pad3)
- RV1 pad 1: +3V3 -> vref2.5
- RV2 pad 1: +3V3 -> vref2.5
- U2 pad 41: amp_control -> usb_sense
- U2 pad 43: +3V3 -> vref2.5
- U5 pad 1: unconnected-(U5-Pad1) -> Net-(R11-Pad2)
- U5 pad 2: Net-(D52-Pad1) -> Net-(J5-Pad2)
- U5 pad 3: Net-(D52-Pad2) -> Net-(J5-Pad3)
- U5 pad 4: unconnected-(U5-Pad4) -> Net-(R21-Pad2)
- U5 pad 7: unconnected-(U5-Pad7) -> /MIDI_RX
Routing:
- net 3v3_filter: track 0.00 -> 421.1 mm, vias 0 -> 25
- net Net-(C10-Pad1): track 391.1 -> 0.00 mm, vias 23 -> 0
- net vref2.5: track 0.00 -> 64.8 mm, vias 0 -> 4
- net +3V3: track 192.2 -> 142.6 mm, vias 11 -> 12
- net Net-(C50-Pad1): track 0.00 -> 47.6 mm, vias 0 -> 3
- net VBUS: track 113.9 -> 79.0 mm, vias 8 -> 7
- net Net-(J5-Pad2): track 0.00 -> 23.8 mm, vias 0 -> 3
- net GND: track 192.4 -> 214.6 mm, vias 24 -> 29
- net Net-(D52-Pad2): track 19.1 -> 0.00 mm, vias 1 -> 0
- net Net-(C4-Pad1): track 16.8 -> 0.00 mm, vias 1 -> 0
- net Net-(JP7-Pad1): track 0.00 -> 13.8 mm, vias 0 -> 2
- net Net-(J3-Pad3): track 16.5 -> 5.74 mm, vias 0 -> 1
- net Net-(C44-Pad2): track 17.5 -> 7.56 mm, vias 1 -> 0
- net usb_sense: track 0.00 -> 9.93 mm, vias 0 -> 2
- net headphone_detect: track 19.7 -> 27.8 mm
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Other:
- board text added: "V10"
- board text removed: "V9"
