File: Hardware/kicad_project/Screen.kicad_sch (KiCad schematic)
At the start: 10 parts, among them U10 apx804SR

Commit message: v9 hardware
Parts:
- removed U10: apx804SR, TO_SOT_Packages_SMD:SOT-23, symbol customLibrary:apx804SR
Changed lines of the file:
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@@
   (junction (at 118.11 109.22) (diameter 0) (color 0 0 0 0)
-  )
-  (junction (at 111.76 99.06) (diameter 0) (color 0 0 0 0)
   )
   (junction (at 118.11 96.52) (diameter 0) (color 0 0 0 0)
@@
     (stroke (width 0) (type default) (color 0 0 0 0))
   )
-  (wire (pts (xy 111.76 99.06) (xy 109.22 99.06))
-    (stroke (width 0) (type default) (color 0 0 0 0))
-  )
   (wire (pts (xy 133.35 109.22) (xy 118.11 109.22))
     (stroke (width 0) (type default) (color 0 0 0 0))
@@
   )
   (wire (pts (xy 118.11 93.98) (xy 154.94 93.98))
-    (stroke (width 0) (type default) (color 0 0 0 0))
-  )
-  (wire (pts (xy 111.76 81.28) (xy 111.76 99.06))
     (stroke (width 0) (type default) (color 0 0 0 0))
   )
@@
     (stroke (width 0) (type default) (color 0 0 0 0))
   )
-  (wire (pts (xy 90.17 81.28) (xy 90.17 78.74))
-    (stroke (width 0) (type default) (color 0 0 0 0))
-  )
   (wire (pts (xy 118.11 96.52) (xy 118.11 106.68))
     (stroke (width 0) (type default) (color 0 0 0 0))
   )
-  (wire (pts (xy 111.76 99.06) (xy 154.94 99.06))
+  (wire (pts (xy 109.22 99.06) (xy 154.94 99.06))
     (stroke (width 0) (type default) (color 0 0 0 0))
   )
@@
     (stroke (width 0) (type default) (color 0 0 0 0))
   )
-  (wire (pts (xy 90.17 83.82) (xy 90.17 85.09))
-    (stroke (width 0) (type default) (color 0 0 0 0))
-  )
   (wire (pts (xy 132.08 83.82) (xy 132.08 86.36))
     (stroke (width 0) (type default) (color 0 0 0 0))
@@
     (stroke (width 0) (type default) (color 0 0 0 0))
   )
-  (wire (pts (xy 95.25 83.82) (xy 90.17 83.82))
-    (stroke (width 0) (type default) (color 0 0 0 0))
-  )
   (wire (pts (xy 137.16 81.28) (xy 154.94 81.28))
-    (stroke (width 0) (type default) (color 0 0 0 0))
-  )
-  (wire (pts (xy 95.25 81.28) (xy 90.17 81.28))
     (stroke (width 0) (type default) (color 0 0 0 0))
   )
@@
     (effects (font (size 1.27 1.27)) (justify right))
   )
-  (symbol (lib_id "Jumper:SolderJumper_2_Bridged") (at 105.41 99.06 0) (mirror y)
+  (symbol (lib_id "Jumper:SolderJumper_2_Bridged") (at 105.41 99.06 0) (mirror y) (unit 1)
     (in_bom yes) (on_board yes)
     (property "Reference" "JP5" (id 0) (at 105.41 93.853 0))
@@
     (pin "2")
   )
-  (symbol (lib_id "customLibrary:apx804SR") (at 102.87 82.55 0) (mirror y)
-    (in_bom yes) (on_board yes)
-    (property "Reference" "U10" (id 0) (at 103.505 74.549 0))
-    (property "Value" "apx804SR" (id 1) (at 103.505 76.8604 0))
-    (property "Footprint" "TO_SOT_Packages_SMD:SOT-23" (id 2) (at 102.87 74.93 0)
-      (effects (font (size 1.27 1.27)) hide)
-    )
-    (property "Datasheet" "" (id 3) (at 102.87 74.93 0)
-      (effects (font (size 1.27 1.27)) hide)
-    )
-    (pin "1")
-    (pin "2")
-    (pin "3")
-  )
-  (symbol (lib_id "power:GND") (at 90.17 85.09 0) (mirror y)
-    (in_bom yes) (on_board yes)
-    (property "Reference" "#PWR0118" (id 0) (at 90.17 91.44 0)
-      (effects (font (size 1.27 1.27)) hide)
-    )
-    (property "Value" "GND" (id 1) (at 90.043 89.4842 0))
-    (property "Footprint" "" (id 2) (at 90.17 85.09 0)
-      (effects (font (size 1.27 1.27)) hide)
-    )
-    (property "Datasheet" "" (id 3) (at 90.17 85.09 0)
-      (effects (font (size 1.27 1.27)) hide)
-    )
-    (pin "1")
-  )
-  (symbol (lib_id "power:+3.3V") (at 90.17 78.74 0) (mirror y)
-    (in_bom yes) (on_board yes)
-    (property "Reference" "#PWR0119" (id 0) (at 90.17 82.55 0)
-      (effects (font (size 1.27 1.27)) hide)
-    )
-    (property "Value" "+3.3V" (id 1) (at 89.789 74.3458 0))
-    (property "Footprint" "" (id 2) (at 90.17 78.74 0)
-      (effects (font (size 1.27 1.27)) hide)
-    )
-    (property "Datasheet" "" (id 3) (at 90.17 78.74 0)
-      (effects (font (size 1.27 1.27)) hide)
-    )
-    (pin "1")
-  )
   (symbol (lib_id "customLibrary:128x32OLED") (at 165.1 95.25 0) (unit 1)

Commit message: v10 board
Parts:
- C51, C52, C53, C54, C55, C56: footprint Capacitors_SMD:C_0402_NoSilk -> Capacitor_SMD:C_0402_1005Metric; checked (none) -> 1
- JP5, LCD1: checked 1 -> (none)
- R15: footprint Resistors_SMD:R_0402_NoSilk -> Resistor_SMD:R_0402_1005Metric; checked (none) -> 1
Connections:
- net +3V3 renamed 3v3_filter
Changed lines of the file:
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@@
   (junction (at 118.11 109.22) (diameter 0) (color 0 0 0 0)
   )
+  (junction (at 129.54 88.9) (diameter 0) (color 0 0 0 0)
+  )
   (junction (at 118.11 96.52) (diameter 0) (color 0 0 0 0)
   )
-  (junction (at 129.54 88.9) (diameter 0) (color 0 0 0 0)
-  )
   (junction (at 118.11 106.68) (diameter 0) (color 0 0 0 0)
   )
@@
     (stroke (width 0) (type default) (color 0 0 0 0))
   )
-  (wire (pts (xy 129.54 88.9) (xy 128.27 88.9))
+  (wire (pts (xy 128.27 88.9) (xy 129.54 88.9))
     (stroke (width 0) (type default) (color 0 0 0 0))
   )
@@
     (stroke (width 0) (type default) (color 0 0 0 0))
   )
+  (wire (pts (xy 129.54 88.9) (xy 154.94 88.9))
+    (stroke (width 0) (type default) (color 0 0 0 0))
+  )
   (wire (pts (xy 154.94 106.68) (xy 149.86 106.68))
     (stroke (width 0) (type default) (color 0 0 0 0))
@@
     (stroke (width 0) (type default) (color 0 0 0 0))
   )
-  (wire (pts (xy 154.94 88.9) (xy 129.54 88.9))
-    (stroke (width 0) (type default) (color 0 0 0 0))
-  )
   (wire (pts (xy 118.11 93.98) (xy 154.94 93.98))
     (stroke (width 0) (type default) (color 0 0 0 0))
@@
     (stroke (width 0) (type default) (color 0 0 0 0))
   )
+  (wire (pts (xy 129.54 73.66) (xy 129.54 88.9))
+    (stroke (width 0) (type default) (color 0 0 0 0))
+  )
   (wire (pts (xy 132.08 83.82) (xy 132.08 86.36))
     (stroke (width 0) (type default) (color 0 0 0 0))
@@
   )
   (wire (pts (xy 137.16 81.28) (xy 154.94 81.28))
-    (stroke (width 0) (type default) (color 0 0 0 0))
-  )
-  (wire (pts (xy 129.54 83.82) (xy 129.54 88.9))
     (stroke (width 0) (type default) (color 0 0 0 0))
   )
@@
     )
   )
+  (global_label "3v3_filter" (shape input) (at 129.54 73.66 180) (fields_autoplaced)
+    (effects (font (size 1.27 1.27)) (justify right))
+    (property "Intersheet References" "${INTERSHEET_REFS}" (id 0) (at 118.2653 73.7394 0)
+      (effects (font (size 1.27 1.27)) (justify right) hide)
+    )
+  )
   (global_label "sda" (shape input) (at 154.94 104.14 180) (fields_autoplaced)
     (effects (font (size 1.27 1.27)) (justify right))
@@
       (effects (font (size 1.27 1.27)) hide)
     )
-    (property "checked" "1" (id 4) (at 105.41 99.06 0)
+    (property "checked" "" (id 4) (at 105.41 99.06 0)
       (effects (font (size 1.27 1.27)) hide)
     )
@@
       (effects (font (size 1.27 1.27)) hide)
     )
-    (property "checked" "1" (id 4) (at 165.1 95.25 0)
+    (property "checked" "" (id 4) (at 165.1 95.25 0)
       (effects (font (size 1.27 1.27)) hide)
     )
@@
       (effects (font (size 1.27 1.27)) (justify left))
     )
-    (property "Footprint" "Capacitors_SMD:C_0402_NoSilk" (id 2) (at 142.24 79.7052 0)
-      (effects (font (size 1.27 1.27)) hide)
-    )
-    (property "Datasheet" "" (id 3) (at 146.05 78.74 0)
+    (property "Footprint" "Capacitor_SMD:C_0402_1005Metric" (id 2) (at 142.24 79.7052 0)
+      (effects (font (size 1.27 1.27)) hide)
+    )
+    (property "Datasheet" "~" (id 3) (at 146.05 78.74 0)
       (effects (font (size 1.27 1.27)) hide)
     )
@@
       (effects (font (size 1.27 1.27)) hide)
     )
+    (property "checked" "1" (id 5) (at 146.05 78.74 0)
+      (effects (font (size 1.27 1.27)) hide)
+    )
     (pin "1")
     (pin "2")
@@
       (effects (font (size 1.27 1.27)) (justify left))
     )
-    (property "Footprint" "Capacitors_SMD:C_0402_NoSilk" (id 2) (at 134.62 84.7852 0)
+    (property "Footprint" "Capacitor_SMD:C_0402_1005Metric" (id 2) (at 134.62 84.7852 0)
       (effects (font (size 1.27 1.27)) hide)
     )
@@
       (effects (font (size 1.27 1.27)) hide)
     )
+    (property "checked" "1" (id 5) (at 138.43 83.82 0)
+      (effects (font (size 1.27 1.27)) hide)
+    )
     (pin "1")
     (pin "2")
@@
       (effects (font (size 1.27 1.27)) (justify left))
     )
-    (property "Footprint" "Capacitors_SMD:C_0402_NoSilk" (id 2) (at 120.65 89.8652 0)
+    (property "Footprint" "Capacitor_SMD:C_0402_1005Metric" (id 2) (at 120.65 89.8652 0)
       (effects (font (size 1.27 1.27)) hide)
     )
@@
       (effects (font (size 1.27 1.27)) hide)
     )
+    (property "checked" "1" (id 5) (at 124.46 88.9 0)
+      (effects (font (size 1.27 1.27)) hide)
+    )
     (pin "1")
     (pin "2")
@@
       (effects (font (size 1.27 1.27)) (justify left))
     )
-    (property "Footprint" "Capacitors_SMD:C_0402_NoSilk" (id 2) (at 120.65 97.4852 0)
+    (property "Footprint" "Capacitor_SMD:C_0402_1005Metric" (id 2) (at 120.65 97.4852 0)
       (effects (font (size 1.27 1.27)) hide)
     )
@@
       (effects (font (size 1.27 1.27)) hide)
     )
-    (pin "1")
-    (pin "2")
-  )
-  (symbol (lib_id "power:+3.3V") (at 129.54 83.82 0) (unit 1)
-    (in_bom yes) (on_board yes)
-    (property "Reference" "#PWR039" (id 0) (at 129.54 87.63 0)
-      (effects (font (size 1.27 1.27)) hide)
-    )
-    (property "Value" "+3.3V" (id 1) (at 129.921 79.4258 0))
-    (property "Footprint" "" (id 2) (at 129.54 83.82 0)
-      (effects (font (size 1.27 1.27)) hide)
-    )
-    (property "Datasheet" "" (id 3) (at 129.54 83.82 0)
-      (effects (font (size 1.27 1.27)) hide)
-    )
-    (pin "1")
+    (property "checked" "1" (id 5) (at 124.46 96.52 0)
+      (effects (font (size 1.27 1.27)) hide)
+    )
+    (pin "1")
+    (pin "2")
   )
   (symbol (lib_id "power:GND") (at 118.11 116.84 0) (unit 1)
@@
       (effects (font (size 1.27 1.27)) (justify left))
     )
-    (property "Footprint" "Capacitors_SMD:C_0402_NoSilk" (id 2) (at 127 112.7252 0)
+    (property "Footprint" "Capacitor_SMD:C_0402_1005Metric" (id 2) (at 127 112.7252 0)
       (effects (font (size 1.27 1.27)) hide)
     )
@@
       (effects (font (size 1.27 1.27)) hide)
     )
+    (property "checked" "1" (id 5) (at 130.81 111.76 0)
+      (effects (font (size 1.27 1.27)) hide)
+    )
     (pin "1")
     (pin "2")
@@
       (effects (font (size 1.27 1.27)) (justify left))
     )
-    (property "Footprint" "Capacitors_SMD:C_0402_NoSilk" (id 2) (at 133.35 110.1852 0)
+    (property "Footprint" "Capacitor_SMD:C_0402_1005Metric" (id 2) (at 133.35 110.1852 0)
       (effects (font (size 1.27 1.27)) hide)
     )
@@
     )
     (property "LCSC" "C15525" (id 4) (at 137.16 109.22 0)
+      (effects (font (size 1.27 1.27)) hide)
+    )
+    (property "checked" "1" (id 5) (at 137.16 109.22 0)
       (effects (font (size 1.27 1.27)) hide)
     )
@@
     (property "Reference" "R15" (id 0) (at 146.05 101.4222 90))
     (property "Value" "330k" (id 1) (at 146.05 103.7336 90))
-    (property "Footprint" "Resistors_SMD:R_0402_NoSilk" (id 2) (at 146.05 104.902 90)
+    (property "Footprint" "Resistor_SMD:R_0402_1005Metric" (id 2) (at 146.05 104.902 90)
       (effects (font (size 1.27 1.27)) hide)
     )
@@
       (effects (font (size 1.27 1.27)) hide)
     )
+    (property "checked" "1" (id 5) (at 146.05 106.68 0)
+      (effects (font (size 1.27 1.27)) hide)
+    )

Commit message: v11 hardware
Connections:
- net 3v3_filter: now also C54.1, LCD1.8 (VDD)
Other:
- moved on the sheet: C53, C54, JP5
