File: Hardware/kicad_project/Power.kicad_sch (KiCad schematic)
At the start: 28 parts, among them J7 battery, J8 Conn_01x03_Male, Q1 DMG2305UX-13, Q2 Q_PMOS_GSD, Q3 Q_NMOS_GSD, Q4 Q_NMOS_GSD, SW1 spst_4_pin_internal, U11 ME6211C, U6 MCP73831T-2ATI_OT

Commit message: v9 hardware
Parts:
- removed J8: Conn_01x03_Male, Connector_PinHeader_2.54mm:PinHeader_1x03_P2.54mm_Horizontal, symbol Connector:Conn_01x03_Male
- D53: LCSC c14996 -> C14996
- D54: LCSC c2286 -> C2286
- SW1: footprint RandomJunk:ts1102_smallerpads_buttonhole -> MyLibrary:ts1187; LCSC C480275 -> C318884
Changed lines of the file:
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@@
   (junction (at 73.66 80.01) (diameter 0) (color 0 0 0 0)
   )
-  (junction (at 172.72 133.35) (diameter 0) (color 0 0 0 0)
-  )
   (junction (at 222.25 87.63) (diameter 0) (color 0 0 0 0)
   )
@@
   (junction (at 146.05 68.58) (diameter 0) (color 0 0 0 0)
   )
-  (junction (at 163.83 111.76) (diameter 0) (color 0 0 0 0)
-  )
   (junction (at 124.46 58.42) (diameter 0) (color 0 0 0 0)
   )
@@
     (stroke (width 0) (type default) (color 0 0 0 0))
   )
-  (wire (pts (xy 172.72 133.35) (xy 163.83 133.35))
+  (wire (pts (xy 163.83 133.35) (xy 182.88 133.35))
     (stroke (width 0) (type default) (color 0 0 0 0))
   )
@@
     (stroke (width 0) (type default) (color 0 0 0 0))
   )
-  (wire (pts (xy 175.26 111.76) (xy 175.26 118.11))
-    (stroke (width 0) (type default) (color 0 0 0 0))
-  )
   (wire (pts (xy 153.67 133.35) (xy 163.83 133.35))
     (stroke (width 0) (type default) (color 0 0 0 0))
@@
     (stroke (width 0) (type default) (color 0 0 0 0))
   )
-  (wire (pts (xy 163.83 111.76) (xy 163.83 115.57))
+  (wire (pts (xy 163.83 109.22) (xy 163.83 115.57))
     (stroke (width 0) (type default) (color 0 0 0 0))
   )
@@
     (stroke (width 0) (type default) (color 0 0 0 0))
   )
-  (wire (pts (xy 172.72 120.65) (xy 172.72 133.35))
-    (stroke (width 0) (type default) (color 0 0 0 0))
-  )
   (wire (pts (xy 156.21 86.36) (xy 156.21 104.14))
     (stroke (width 0) (type default) (color 0 0 0 0))
@@
     (stroke (width 0) (type default) (color 0 0 0 0))
   )
-  (wire (pts (xy 163.83 111.76) (xy 175.26 111.76))
-    (stroke (width 0) (type default) (color 0 0 0 0))
-  )
   (wire (pts (xy 203.2 68.58) (xy 209.55 68.58))
     (stroke (width 0) (type default) (color 0 0 0 0))
@@
     (stroke (width 0) (type default) (color 0 0 0 0))
   )
-  (wire (pts (xy 175.26 120.65) (xy 172.72 120.65))
-    (stroke (width 0) (type default) (color 0 0 0 0))
-  )
   (wire (pts (xy 209.55 87.63) (xy 222.25 87.63))
     (stroke (width 0) (type default) (color 0 0 0 0))
@@
     (stroke (width 0) (type default) (color 0 0 0 0))
   )
-  (wire (pts (xy 182.88 133.35) (xy 172.72 133.35))
-    (stroke (width 0) (type default) (color 0 0 0 0))
-  )
   (wire (pts (xy 96.52 123.19) (xy 96.52 115.57))
     (stroke (width 0) (type default) (color 0 0 0 0))
   )
   (wire (pts (xy 173.99 76.2) (xy 173.99 104.14))
-    (stroke (width 0) (type default) (color 0 0 0 0))
-  )
-  (wire (pts (xy 163.83 109.22) (xy 163.83 111.76))
     (stroke (width 0) (type default) (color 0 0 0 0))
   )
@@
     (pin "3")
   )
-  (symbol (lib_id "customLibrary:spst_4_pin_internal") (at 162.56 120.65 270)
+  (symbol (lib_id "customLibrary:spst_4_pin_internal") (at 162.56 120.65 270) (unit 1)
     (in_bom yes) (on_board yes)
     (property "Reference" "SW1" (id 0) (at 172.466 120.65 0))
     (property "Value" "spst_4_pin_internal" (id 1) (at 170.1546 120.65 0))
-    (property "Footprint" "RandomJunk:ts1102_smallerpads_buttonhole" (id 2) (at 162.56 121.92 0)
+    (property "Footprint" "MyLibrary:ts1187" (id 2) (at 162.56 121.92 0)
       (effects (font (size 1.27 1.27)) hide)
     )
@@
       (effects (font (size 1.27 1.27)) hide)
     )
-    (property "LCSC" "C480275" (id 4) (at 162.56 120.65 0)
+    (property "LCSC" "C318884" (id 4) (at 162.56 120.65 0)
       (effects (font (size 1.27 1.27)) hide)
     )
@@
     (pin "2")
   )
-  (symbol (lib_id "Jumper:SolderJumper_2_Bridged") (at 133.35 86.36 0)
+  (symbol (lib_id "Jumper:SolderJumper_2_Bridged") (at 133.35 86.36 0) (unit 1)
     (in_bom yes) (on_board yes)
     (property "Reference" "JP6" (id 0) (at 133.35 81.153 0))
@@
     (pin "2")
   )
-  (symbol (lib_id "Connector:Conn_01x03_Male") (at 180.34 120.65 180) (unit 1)
-    (in_bom yes) (on_board yes)
-    (property "Reference" "J8" (id 0) (at 181.0512 118.9228 0)
-      (effects (font (size 1.27 1.27)) (justify right))
-    )
-    (property "Value" "Conn_01x03_Male" (id 1) (at 181.0512 121.2342 0)
-      (effects (font (size 1.27 1.27)) (justify right))
-    )
-    (property "Footprint" "Connector_PinHeader_2.54mm:PinHeader_1x03_P2.54mm_Horizontal" (id 2) (at 180.34 120.65 0)
-      (effects (font (size 1.27 1.27)) hide)
-    )
-    (property "Datasheet" "~" (id 3) (at 180.34 120.65 0)
-      (effects (font (size 1.27 1.27)) hide)
-    )
-    (property "checked" "1" (id 4) (at 180.34 120.65 0)
-      (effects (font (size 1.27 1.27)) hide)
-    )
-    (pin "1")
-    (pin "2")
-    (pin "3")
-  )
   (symbol (lib_id "power:+BATT") (at 143.51 50.8 0) (unit 1)
     (in_bom yes) (on_board yes)
@@
       (effects (font (size 1.27 1.27)) hide)
     )
-    (property "LCSC" "c14996" (id 4) (at 128.27 68.58 0)
+    (property "LCSC" "C14996" (id 4) (at 128.27 68.58 0)
       (effects (font (size 1.27 1.27)) hide)
     )
@@
       (effects (font (size 1.27 1.27)) hide)
     )
-    (property "LCSC" "c2286" (id 4) (at 95.25 72.39 0)
-      (effects (font (size 1.27 1.27)) hide)
-    )
+    (property "LCSC" "C2286" (id 4) (at 95.25 72.39 0)
+      (effects (font (size 1.27 1.27)) hide)
+    )

Commit message: v10 board
Parts:
- added C50: 10u, Capacitor_SMD:C_0402_1005Metric, symbol Device:C
- added C65: 100u, Capacitor_Tantalum_SMD:CP_EIA-3528-21_Kemet-B, symbol Device:C
- added J8: Conn_01x02_Female, Connector_PinHeader_2.54mm:PinHeader_1x02_P2.54mm_Vertical, symbol Connector:Conn_01x02_Female
- added JP7, JP8: SolderJumper_2_Bridged, Jumper:SolderJumper-2_P1.3mm_Bridged_Pad1.0x1.5mm, symbol Jumper:SolderJumper_2_Bridged
- added R22: 330, Resistor_SMD:R_0402_1005Metric, symbol Device:R_US
- added R23: 5k, Resistor_SMD:R_0402_1005Metric, symbol Device:R_US
- added R30: 10k, Resistor_SMD:R_0402_1005Metric, symbol Device:R_US
- added R34, R35: 33, Resistor_SMD:R_0402_1005Metric, symbol Device:R
- added U7: LM4040DBZ-2.5, Package_TO_SOT_SMD:SOT-23, symbol Reference_Voltage:LM4040DBZ-2.5
- C57, C59, C60, C61, C62, C64: footprint Capacitors_SMD:C_0402_NoSilk -> Capacitor_SMD:C_0402_1005Metric; checked (none) -> 1
- D1, D53, D54, Q2, Q3, Q4, R29, SW1: checked (none) -> 1
- JP6: checked 1 -> (none)
- Q1: Category Discrete Semiconductor Products -> (none); DK_Datasheet_Link https://www.diodes.com/assets/Datasheets/DMG2305UX.pdf -> (none); DK_Detail_Page /product-detail/en/diodes-incorporated/DMG2305UX-13/DMG2305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 -> (none); Digi-Key_PN DMG2305UX-13DICT-ND -> (none); Family Transistors - FETs, MOSFETs - Single -> (none); LCSC C144153 -> C2940629; MPN DMG2305UX-13 -> (none); Manufacturer Diodes Incorporated -> (none); Status Active -> (none); checked (none) -> 1
- R16, R17, R18, R25, R26, R27, R28, R8: footprint Resistors_SMD:R_0402_NoSilk -> Resistor_SMD:R_0402_1005Metric; checked (none) -> 1
- U6: DK_Datasheet_Link http://ww1.microchip.com/downloads/en/DeviceDoc/20001984g.p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 -> (none); DK_Detail_Page /product-detail/en/microchip-technology/MCP73831T-2ATI-OT/M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 -> (none); Digi-Key_PN MCP73831T-2ATI/OTCT-ND -> (none); Family PMIC - Battery Chargers -> (none); MPN MCP73831T-2ATI/OT -> (none); Manufacturer Microchip Technology -> (none); Status Active -> (none)
Connections:
- net +3V3: now also J8.2 (Pin_2), R34.1, R35.1
- net GND: now also C50.2, C65.2, R30.1, U7.2 (A)
- net VBUS: now also R22.2, R23.2
- new net: C50.1, C65.1, J8.1 (Pin_1), JP7.2 (B), JP8.1 (A)
- new net: JP7.1 (A), R34.2, R35.2
- new net 3v3_filter: JP8.2 (B)
- new net usb_sense: R23.1, R30.2
- new net vref2.5: R22.1, U7.1 (K)
Other:
- note added: "RC filtered power for screen & LEDs"
- note added: "input range voltage 3-5.1 from battery or usb"
- moved on the sheet: C57, C59, C60, C61, C62, C64, D1, D53, D54, J7, JP6, Q1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

Commit message: v11 hardware
Parts:
- R23: value 5k -> 5.1k; LCSC C477765 -> C25905
Connections:
- net VBUS: no longer C60.1, C64.1, Q2.3 (D), U11.1 (IN), U11.3 (~{EN})
- new net VSYS: C60.1, C64.1, Q2.3 (D), U11.1 (IN), U11.3 (~{EN})
Changed lines of the file:
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@@
     (pin "2")
   )
-  (symbol (lib_id "customLibrary:VSYS") (at 218.44 49.53 0) (unit 1)
+  (symbol (lib_name "VSYS_1") (lib_id "customLibrary:VSYS") (at 218.44 49.53 0) (unit 1)
     (in_bom yes) (on_board yes)
     (property "Reference" "#PWR0126" (id 0) (at 218.44 53.34 0)
@@
     (in_bom yes) (on_board yes)
     (property "Reference" "R23" (id 0) (at 86.487 101.6 90))
-    (property "Value" "5k" (id 1) (at 84.1756 101.6 90))
+    (property "Value" "5.1k" (id 1) (at 84.1756 101.6 90))
     (property "Footprint" "Resistor_SMD:R_0402_1005Metric" (id 2) (at 80.264 101.346 90)
       (effects (font (size 1.27 1.27)) hide)
@@
       (effects (font (size 1.27 1.27)) hide)
     )
-    (property "LCSC" "C477765" (id 4) (at 81.28 101.6 0)
-      (effects (font (size 1.27 1.27)) hide)
-    )
+    (property "LCSC" "C25905" (id 4) (at 81.28 101.6 0)
+      (effects (font (size 1.27 1.27)) hide)
+    )

Commit message: pcb bodge fixes
Connections:
- net VBUS: no longer R22.2
- net VSYS: now also R22.2
Changed lines of the file:
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@@
     (pin "2")
-  )
-  (symbol (lib_id "customLibrary:VSYS") (at 109.22 88.9 0) (unit 1)
-    (in_bom yes) (on_board yes)
-    (property "Reference" "#PWR0132" (id 0) (at 109.22 92.71 0)
-      (effects (font (size 1.27 1.27)) hide)
-    )
-    (property "Value" "VSYS" (id 1) (at 109.601 84.5058 0))
-    (property "Footprint" "" (id 2) (at 109.22 88.9 0)
-      (effects (font (size 1.27 1.27)) hide)
-    )
-    (property "Datasheet" "" (id 3) (at 109.22 88.9 0)
-      (effects (font (size 1.27 1.27)) hide)
-    )
-    (pin "1")
   )
   (symbol (lib_id "Device:R_US") (at 81.28 101.6 180) (unit 1)
@@
       (effects (font (size 1.27 1.27)) hide)
     )
+    (pin "1")
+  )
+  (symbol (lib_name "VSYS_1") (lib_id "customLibrary:VSYS") (at 109.22 88.9 0) (unit 1)
+    (in_bom yes) (on_board yes)
+    (property "Reference" "#PWR0132" (id 0) (at 109.22 92.71 0)
+      (effects (font (size 1.27 1.27)) hide)
+    )
+    (property "Value" "VSYS" (id 1) (at 109.601 84.5058 0))
+    (property "Footprint" "" (id 2) (at 109.22 88.9 0)
+      (effects (font (size 1.27 1.27)) hide)
+    )
+    (property "Datasheet" "" (id 3) (at 109.22 88.9 0)
+      (effects (font (size 1.27 1.27)) hide)
+    )
