File: Enclosure/frontplate/frontplate.kicad_pcb (KiCad board)
At the start: 2 copper layers, 65 x 100 mm, 8 parts

Commit message: v9 hardware
Parts:
- removed the G*** at (64.5, 83.0)
- moved G*** 0.30 mm to (64.5, 82.7)
- moved G*** 0.28 mm to (64.5, 82.7)
Routing:
- added copper zone on B.Cu, net (none)
- added copper zone on F.Cu, net (none)
Other:
- outline, holes or cut-outs redrawn
- net class Default removed
- rule pad_to_mask_clearance: 0.051 -> 0

Commit message: new faceplate
Parts:
- added REF**: LargeButtonHole, MyLibrary:LargeButtonHole, F.Cu at (42.5, 86.7)
- added REF**1: LargeButtonHole, MyLibrary:LargeButtonHole, F.Cu at (53.5, 86.7)
- added REF**10: LargeButtonHole, MyLibrary:LargeButtonHole, F.Cu at (42.5, 110.7)
- added REF**11: LargeButtonHole, MyLibrary:LargeButtonHole, F.Cu at (53.5, 110.7)
- added REF**12: LargeButtonHole, MyLibrary:LargeButtonHole, F.Cu at (64.5, 110.7)
- added REF**13: LargeButtonHole, MyLibrary:LargeButtonHole, F.Cu at (75.5, 110.7)
- added REF**14: LargeButtonHole, MyLibrary:LargeButtonHole, F.Cu at (86.5, 110.7)
- added REF**15: LargeButtonHole, MyLibrary:LargeButtonHole, F.Cu at (42.5, 122.7)
- added REF**16: LargeButtonHole, MyLibrary:LargeButtonHole, F.Cu at (53.5, 122.7)
- added REF**17: LargeButtonHole, MyLibrary:LargeButtonHole, F.Cu at (64.5, 122.7)
- added REF**18: LargeButtonHole, MyLibrary:LargeButtonHole, F.Cu at (75.5, 122.7)
- added REF**19: LargeButtonHole, MyLibrary:LargeButtonHole, F.Cu at (86.5, 122.7)
- added REF**2: LargeButtonHole, MyLibrary:LargeButtonHole, F.Cu at (64.5, 86.7)
- added REF**3: LargeButtonHole, MyLibrary:LargeButtonHole, F.Cu at (75.5, 86.7)
- added REF**4: LargeButtonHole, MyLibrary:LargeButtonHole, F.Cu at (86.5, 86.7)
- added REF**5: LargeButtonHole, MyLibrary:LargeButtonHole, F.Cu at (42.5, 98.7)
- added REF**6: LargeButtonHole, MyLibrary:LargeButtonHole, F.Cu at (53.5, 98.7)
- added REF**7: LargeButtonHole, MyLibrary:LargeButtonHole, F.Cu at (64.5, 98.7)
- added REF**8: LargeButtonHole, MyLibrary:LargeButtonHole, F.Cu at (75.5, 98.7)
- added REF**9: LargeButtonHole, MyLibrary:LargeButtonHole, F.Cu at (86.5, 98.7)
Other:
- outline, holes or cut-outs redrawn
