File: Hardware/audcalc/ButtonsLEDS.kicad_sch (KiCad schematic)
At the start: 89 parts, among them SW10 spst_4_pin_internal, SW11 spst_4_pin_internal, SW12 spst_4_pin_internal, SW13 spst_4_pin_internal, SW14 spst_4_pin_internal, SW15 spst_4_pin_internal, SW16 spst_4_pin_internal, SW17 spst_4_pin_internal, SW18 spst_4_pin_internal, SW19 spst_4_pin_internal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

Commit message: update schematic doc block
Other:
- company: TWR -> Jonathan Brodsky
- title: TDM -> Aud Calc
Changed lines of the file:
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@@
 	(paper "A4")
 	(title_block
-		(title "TDM")
-		(date "2021-09-17")
-		(rev "6")
-		(company "TWR")
-		(comment 1 "Pocket Sound Computer")
+		(title "Aud Calc")
+		(date "2024-04-04")
+		(rev "12")
+		(company "Jonathan Brodsky")
+		(comment 1 "Pocket Sound Calculator")
 	)
 	(junction
