File: Hardware/audcalc/ButtonsLEDS.kicad_sch (KiCad schematic)
At the start: 89 parts, among them SW10 spst_4_pin_internal, SW11 spst_4_pin_internal, SW12 spst_4_pin_internal, SW13 spst_4_pin_internal, SW14 spst_4_pin_internal, SW15 spst_4_pin_internal, SW16 spst_4_pin_internal, SW17 spst_4_pin_internal, SW18 spst_4_pin_internal, SW19 spst_4_pin_internal, SW2 spst_4_pin_internal, SW20 spst_4_pin_internal, SW21 spst_4_pin_internal, SW22 spst_4_pin_internal, SW23 spst_4_pin_internal, SW24 spst_4_pin_internal, SW25 spst_4_pin_internal, SW3 spst_4_pin_internal, SW4 spst_4_pin_internal, SW5 spst_4_pin_internal, SW6 spst_4_pin_internal, SW7 spst_4_pin_internal, SW8 spst_4_pin_internal, SW9 spst_4_pin_internal

Commit message: updated PCB with new JLC part numbers
Parts:
- C10, C11, C12, C13, C14, C15, C16, C17, C18, C19, C20, C21, C22, C23, C24, C25, C6, C7, C8, C9: footprint Capacitor_SMD:C_0402_1005Metric -> MyLibrary:C_0402_1005Metric
