File: Hardware/audcalc/Screen.kicad_sch (KiCad schematic)
At the start: 9 parts

Commit message: update schematic doc block
Other:
- company: TWR -> Jonathan Brodsky
- title: TDM -> Aud Calc
Changed lines of the file:
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@@
 	(paper "A4")
 	(title_block
-		(title "TDM")
-		(date "2021-09-17")
-		(rev "6")
-		(company "TWR")
-		(comment 1 "Pocket Sound Computer")
+		(title "Aud Calc")
+		(date "2024-04-04")
+		(rev "12")
+		(company "Jonathan Brodsky")
+		(comment 1 "Pocket Sound Calculator")
 	)
 	(junction
