File: Hardware/audcalc/Screen.kicad_sch (KiCad schematic)
At the start: 9 parts

Commit message: updated PCB with new JLC part numbers
Parts:
- C51, C52, C53, C54, C55, C56: footprint Capacitor_SMD:C_0402_1005Metric -> MyLibrary:C_0402_1005Metric
- LCD1: footprint RandomJunk:oled_ssd1306_14pin_91 -> MyLibrary:oled_ssd1306_14pin_91
- R15: footprint Resistor_SMD:R_0402_1005Metric -> MyLibrary:R_0402_1005Metric_nosilk
