File: Hardware/audcalc/Power.kicad_sch (KiCad schematic)
At the start: 38 parts, among them J7 battery, J8 Conn_01x02_Female, Q1 DMG2305UX-13, Q2 Q_PMOS_GSD, Q3 Q_NMOS_GSD, Q4 Q_NMOS_GSD, SW1 spst_4_pin_internal, U11 ME6211C, U6 MCP73831T-2ATI_OT, U7 LM4040DBZ-2.5

Commit message: update schematic doc block
Other:
- company: TWR -> Jonathan Brodsky
- title: TDM -> Aud Calc
Changed lines of the file:
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@@
 	(paper "A4")
 	(title_block
-		(title "TDM")
-		(date "2021-09-17")
-		(rev "6")
-		(company "TWR")
-		(comment 1 "Pocket Sound Computer")
+		(title "Aud Calc")
+		(date "2024-04-04")
+		(rev "12")
+		(company "Jonathan Brodsky")
+		(comment 1 "Pocket Sound Calculator")
 	)
 	(junction
@@
 		)
 		(property "Description" ""
-			(at 76.2 54.61 0)
+			(at 81.28 29.21 0)
 			(effects
 				(font
-					(size 1.27 1.27)
+					(size 1.524 1.524)
 				)
+				(justify left)
 				(hide yes)
 			)
@@
 			)
 		)
-		(property "Description" ""
-			(at 81.28 29.21 0)
-			(effects
-				(font
-					(size 1.524 1.524)
-				)
-				(justify left)
-				(hide yes)
-			)
-		)
 		(property "Manufacturer" ""
 			(at 81.28 26.67 0)
@@
 		)
 		(property "Description" ""
-			(at 172.72 44.45 0)
+			(at 177.8 19.05 0)
 			(effects
 				(font
-					(size 1.27 1.27)
+					(size 1.524 1.524)
 				)
+				(justify left)
 				(hide yes)
 			)
@@
 			(effects
 				(font
-					(size 1.524 1.524)
-				)
-				(justify left)
-				(hide yes)
-			)
-		)
-		(property "Description" ""
-			(at 177.8 19.05 0)
-			(effects
-				(font

Commit message: fixed up bom for JLC
Parts:
- Q1: LCSC C2940629 -> C144153
Changed lines of the file:
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@@
 			)
 		)
-		(property "LCSC" "C2940629"
+		(property "LCSC" "C144153"
 			(at 172.72 44.45 0)
 			(effects
