File: Hardware/audcalc/Power.kicad_sch (KiCad schematic)
At the start: 38 parts, among them J7 battery, J8 Conn_01x02_Female, Q1 DMG2305UX-13, Q2 Q_PMOS_GSD, Q3 Q_NMOS_GSD, Q4 Q_NMOS_GSD, SW1 spst_4_pin_internal, U11 ME6211C, U6 MCP73831T-2ATI_OT, U7 LM4040DBZ-2.5

Commit message: updated PCB with new JLC part numbers
Parts:
- C50, C57, C59, C60, C61, C62, C64: footprint Capacitor_SMD:C_0402_1005Metric -> MyLibrary:C_0402_1005Metric
- J7: LCSC (none) -> C3029440
- R16, R17, R18, R22, R23, R25, R26, R27, R28, R30, R34, R35, R8: footprint Resistor_SMD:R_0402_1005Metric -> MyLibrary:R_0402_1005Metric_nosilk
