File: Hardware/audcalc/audcalc.kicad_pcb (KiCad board)
At the start: 4 copper layers, 65 x 100 mm, 218 parts, among them J1 picoprobe_debug, J2 USB_C_Receptacle_USB2.0, J3 line_in, J4 headphone_out, J5 midi_in, J6 midi_out, J7 battery, J8 Conn_01x02_Female, Q1 DMG2305UX-13, Q2 Q_PMOS_GSD, Q3 Q_NMOS_GSD, Q4 Q_NMOS_GSD, SW1 spst_4_pin_internal, SW10 spst_4_pin_internal, SW11 spst_4_pin_internal, SW12 spst_4_pin_internal, SW13 spst_4_pin_internal, SW14 spst_4_pin_internal, SW15 spst_4_pin_internal, SW16 spst_4_pin_internal, SW17 spst_4_pin_internal, SW18 spst_4_pin_internal, SW19 spst_4_pin_internal, SW2 spst_4_pin_internal, SW20 spst_4_pin_internal, SW21 spst_4_pin_internal, SW22 spst_4_pin_internal, SW23 spst_4_pin_internal, SW24 spst_4_pin_internal, SW25 spst_4_pin_internal, SW26 spst_4_pin_internal, SW27 spst_4_pin_internal, SW3 spst_4_pin_internal, SW4 spst_4_pin_internal, SW5 spst_4_pin_internal, SW6 spst_4_pin_internal, SW7 spst_4_pin_internal, SW8 spst_4_pin_internal, SW9 spst_4_pin_internal, U1 W25Q32JVSS, U11 ME6211C, U2 RP2040, U3 TLV320AIC3204, U4 AP3722AT_mic, U5 HCPL-0631, U6 MCP73831T-2ATI_OT, U7 LM4040DBZ-2.5, U9 ME6211C, Y1 Crystal_GND24

Commit message: fixed up bom for JLC
Parts:
- U4: footprint MyLibrary:LGA-4(3x3.8) -> MyLibrary:LGA-4 (3x3.8)
- turned U4 to 90 degrees
Changed lines of the file:
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@@
 			(drillshape 0)
 			(scaleselection 1)
-			(outputdirectory "../")
+			(outputdirectory "../gerber/")
 		)
 	)
@@
 		)
 	)
-	(footprint "MyLibrary:LGA-4(3x3.8)"
+	(footprint "MyLibrary:LGA-4 (3x3.8)"
 		(layer "F.Cu")
-		(at 88.7 50.6)
+		(at 88.7 50.6 90)
 		(property "Reference" "U4"
-			(at 0 -2.5 0)
+			(at -0.2 -2.7 90)
 			(unlocked yes)
 			(layer "F.SilkS")
+			(hide yes)
 			(effects
 				(font
@@
 		)
 		(property "Value" "AP3722AT_mic"
-			(at 0 2.2 0)
+			(at -0.1 2.5 90)
 			(unlocked yes)
 			(layer "F.Fab")
@@
 		)
 		(property "Footprint" ""
-			(at 0 0 0)
+			(at 0 0 90)
 			(unlocked yes)
 			(layer "F.Fab")
@@
 			(effects
 				(font
-					(size 1.27 1.27)
+					(size 1 1)
+					(thickness 0.15)
 				)
 			)
 		)
 		(property "Datasheet" ""
-			(at 0 0 0)
+			(at 0 0 90)
 			(unlocked yes)
 			(layer "F.Fab")
@@
 			(effects
 				(font
-					(size 1.27 1.27)
+					(size 1 1)
+					(thickness 0.15)
 				)
 			)
 		)
 		(property "Description" ""
-			(at 0 0 0)
+			(at 0 0 90)
 			(unlocked yes)
 			(layer "F.Fab")
@@
 			(effects
 				(font
-					(size 1.27 1.27)
+					(size 1 1)
+					(thickness 0.15)
 				)
 			)
 		)
 		(property "LCSC" "C918198"
-			(at 0 0 0)
+			(at 0 0 270)
 			(layer "F.Fab")
 			(hide yes)
@@
 		)
 		(property "checked" "1"
-			(at 0 0 0)
+			(at 0 0 270)
 			(layer "F.Fab")
 			(hide yes)
@@
 			)
 		)
-		(sheetname "AudioMidi")
-		(sheetfile "audioMidi.kicad_sch")
 		(attr smd)
+		(fp_line
+			(start 0.8 -2.2)
+			(end 1.8 -2.2)
+			(stroke
+				(width 0.12)
+				(type default)
+			)
+			(layer "F.SilkS")
+		)
+		(fp_line
+			(start 1.8 -1.2)
+			(end 1.8 -2.2)
+			(stroke
+				(width 0.12)
+				(type default)
+			)
+			(layer "F.SilkS")
+		)
+		(fp_line
+			(start 1.48 -1.88)
+			(end 1.48 1.88)
+			(stroke
+				(width 0.05)
+				(type default)
+			)
+			(layer "F.CrtYd")
+		)
+		(fp_line
+			(start -1.48 -1.88)
+			(end 1.48 -1.88)
+			(stroke
+				(width 0.05)
+				(type default)
+			)
+			(layer "F.CrtYd")
+		)
+		(fp_line
+			(start 1.48 1.88)
+			(end -1.48 1.88)
+			(stroke
+				(width 0.05)
+				(type default)
+			)
+			(layer "F.CrtYd")
+		)
+		(fp_line
+			(start -1.48 1.88)
+			(end -1.48 -1.88)
+			(stroke
+				(width 0.05)
+				(type default)
+			)
+			(layer "F.CrtYd")
+		)
 		(fp_text user "${REFERENCE}"
-			(at 0 4 0)
+			(at -0.1 4 90)
 			(unlocked yes)
 			(layer "F.Fab")
@@
 		)
 		(pad "1" smd circle
-			(at -1.23 -0.85)
+			(at 0.85 -1.23 90)
 			(size 0.8 0.8)
 			(layers "F.Cu" "F.Paste" "F.Mask")
@@
 		)
 		(pad "2" smd circle
-			(at 1.23 -0.85)
+			(at 0.85 1.23 90)
 			(size 0.8 0.8)
 			(layers "F.Cu" "F.Paste" "F.Mask")
@@
 		)
 		(pad "3" smd circle
-			(at 1.23 0.85)
+			(at -0.85 1.23 90)
 			(size 0.8 0.8)
 			(layers "F.Cu" "F.Paste" "F.Mask")
@@
 		)
 		(pad "4" smd circle
-			(at -1.23 0.85)
+			(at -0.85 -1.23 90)
 			(size 0.8 0.8)
 			(layers "F.Cu" "F.Paste" "F.Mask")
@@
 	)
 	(gr_line
-		(start 86.7 50)
-		(end 86.7 49)
-		(stroke
-			(width 0.12)
-			(type solid)
-		)
-		(layer "F.SilkS")
-	)
-	(gr_line
-		(start 86.7 49)
-		(end 87.7 49)
-		(stroke
-			(width 0.12)
-			(type solid)
-		)
-		(layer "F.SilkS")
-	)
-	(gr_line
