File: Hardware/audcalc/audcalc.kicad_pcb (KiCad board)
At the start: 4 copper layers, 65 x 100 mm, 218 parts, among them J1 picoprobe_debug, J2 USB_C_Receptacle_USB2.0, J3 line_in, J4 headphone_out, J5 midi_in, J6 midi_out, J7 battery, J8 Conn_01x02_Female, Q1 DMG2305UX-13, Q2 Q_PMOS_GSD, Q3 Q_NMOS_GSD, Q4 Q_NMOS_GSD, SW1 spst_4_pin_internal, SW10 spst_4_pin_internal, SW11 spst_4_pin_internal, SW12 spst_4_pin_internal, SW13 spst_4_pin_internal, SW14 spst_4_pin_internal, SW15 spst_4_pin_internal, SW16 spst_4_pin_internal, SW17 spst_4_pin_internal, SW18 spst_4_pin_internal, SW19 spst_4_pin_internal, SW2 spst_4_pin_internal, SW20 spst_4_pin_internal, SW21 spst_4_pin_internal, SW22 spst_4_pin_internal, SW23 spst_4_pin_internal, SW24 spst_4_pin_internal, SW25 spst_4_pin_internal, SW26 spst_4_pin_internal, SW27 spst_4_pin_internal, SW3 spst_4_pin_internal, SW4 spst_4_pin_internal, SW5 spst_4_pin_internal, SW6 spst_4_pin_internal, SW7 spst_4_pin_internal, SW8 spst_4_pin_internal, SW9 spst_4_pin_internal, U1 W25Q32JVSS, U11 ME6211C, U2 RP2040, U3 TLV320AIC3204, U4 AP3722AT_mic, U5 HCPL-0631, U6 MCP73831T-2ATI_OT, U7 LM4040DBZ-2.5, U9 ME6211C, Y1 Crystal_GND24

Commit message: updated PCB with new JLC part numbers
Parts:
- C58: value 10u -> 10u(tant)
- D2: value LEDGreen -> LEDYellow
- SW26, SW27: value spst_4_pin_internal -> spst_4_pin_internal_side
- U4: value AP3722AT_mic -> WMM7037AT2_mic
