File: Hardware/audcalc/audcalc.kicad_sch (KiCad schematic)
At the start: 40 parts, among them J1 picoprobe_debug, J2 USB_C_Receptacle_USB2.0, SW26 spst_4_pin_internal, SW27 spst_4_pin_internal, U1 W25Q32JVSS, U2 RP2040, Y1 Crystal_GND24

Commit message: update schematic doc block
Other:
- company: TWR -> Jonathan Brodsky
- title: TDM -> Aud Calc
Changed lines of the file:
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@@
 	(paper "A4")
 	(title_block
-		(title "TDM")
-		(date "2021-09-17")
-		(rev "6")
-		(company "TWR")
-		(comment 1 "Pocket Sound Computer")
+		(title "Aud Calc")
+		(date "2024-04-04")
+		(rev "12")
+		(company "Jonathan Brodsky")
+		(comment 1 "Pocket Sound Calculator")
 	)
 	(junction

Commit message: fixed up bom for JLC
Parts:
- D2: value LEDGreen -> LEDYellow; LCSC C72043 -> C72038
- SW26, SW27: value spst_4_pin_internal -> spst_4_pin_internal_side
Changed lines of the file:
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@@
 			)
 		)
-		(property "Value" "spst_4_pin_internal"
+		(property "Value" "spst_4_pin_internal_side"
 			(at 97.79 77.4954 0)
 			(effects
@@
 			)
 		)
-		(property "Value" "LEDGreen"
+		(property "Value" "LEDYellow"
 			(at 269.4178 140.335 0)
 			(effects
@@
 			)
 		)
-		(property "LCSC" "C72043"
+		(property "LCSC" "C72038"
 			(at 269.24 137.16 0)
 			(effects
@@
 			)
 		)
-		(property "Value" "spst_4_pin_internal"
+		(property "Value" "spst_4_pin_internal_side"
 			(at 172.72 120.6754 0)
 			(effects
