File: Hardware/audcalc/audcalc.kicad_sch (KiCad schematic)
At the start: 40 parts, among them J1 picoprobe_debug, J2 USB_C_Receptacle_USB2.0, SW26 spst_4_pin_internal_side, SW27 spst_4_pin_internal_side, U1 W25Q32JVSS, U2 RP2040, Y1 Crystal_GND24

Commit message: updated PCB with new JLC part numbers
Parts:
- C1, C2, C26, C27, C28, C29, C3, C30, C31, C32, C33, C34, C35, C36, C37, C66: footprint Capacitor_SMD:C_0402_1005Metric -> MyLibrary:C_0402_1005Metric
- D2: LCSC C72038 -> C89811
- H1, H2, H3, H4: now not fitted
- R1, R19, R2, R20, R3, R31, R6, R7: footprint Resistor_SMD:R_0402_1005Metric -> MyLibrary:R_0402_1005Metric_nosilk
- RV1, RV2: LCSC (none) -> C209779
