File: Hardware/audcalc/audioMidi.kicad_sch (KiCad schematic)
At the start: 42 parts, among them J3 line_in, J4 headphone_out, J5 midi_in, J6 midi_out, U3 TLV320AIC3204, U4 WMM7037AT2_mic, U5 HCPL-0631, U9 ME6211C

Commit message: updated PCB with new JLC part numbers
Parts:
- C38, C4, C40, C41, C42, C43, C46, C5, C63: footprint Capacitor_SMD:C_0402_1005Metric -> MyLibrary:C_0402_1005Metric
- J3, J4, J5, J6: LCSC (none) -> C145813
- R10, R11, R12, R13, R14, R21, R24, R9: footprint Resistor_SMD:R_0402_1005Metric -> MyLibrary:R_0402_1005Metric_nosilk
- R32, R33: footprint Resistor_SMD:R_01005_0402Metric -> Resistor_SMD:R_0402_1005Metric
- U4: footprint MyLibrary:LGA-4(3x3.8) -> MyLibrary:LGA-4 (3x3.8)
